File: atmega328p-base.kicad_pcb (KiCad board)
At the start: 2 copper layers, 43.2 x 43.2 mm, 24 parts, among them J0 ICSP, J1 USB_to_TTL, J31 pins_1_8, J32 pins_8_16, J33 pins_17_24, J34 pins_25_32, U1 ATmega328PB-AU, Y1 16MHz

Commit message: bigger size C, tidy-up
Parts:
- added REF**: mo-logo-small-on-side, meon:mo-logo-small-on-side, B.Cu at (146.1, 125.7)
- C0, C11, C12, C2: footprint Capacitor_SMD:C_0603_1608Metric_Pad1.05x0.95mm_HandSolder_no_lines -> Capacitor_SMD:C_0805_2012Metric_no_lines
- R0: value 10k -> 1k
- REF**: value mo-logo-small -> mo-logo-small-on-side; footprint meon:mo-logo-small -> meon:mo-logo-small-on-side
- moved C11 0.92 mm to (132.8, 138.2)
- moved C12 0.80 mm to (135.4, 138.2)
- moved C2 0.51 mm to (156.5, 114.6)
- moved C0 0.25 mm to (154.7, 125.0), turned to 0 degrees
Routing:
- net D2: track 25.2 -> 17.3 mm
- net GND: track 68.6 -> 71.3 mm
- net VCC: track 145.5 -> 143.7 mm
- net TXD: track 26.7 -> 25.2 mm
- net ~RST: track 106.0 -> 107.2 mm
- net XTAL2: track 36.8 -> 38.0 mm
- net DTR: track 4.15 -> 5.29 mm
- net D12_MISO: track 23.3 -> 22.2 mm
- net XTAL1: track 36.9 -> 37.5 mm
- net AREF: track 16.8 -> 16.3 mm
Other:
- board text added: ">1k"
- board text removed: "100nF"
- board text removed: "1k"
- board text removed: "2x 22pF"
